Commit message: Whole process works

File: src/Universal_Robots_ROS2_Description/urdf/ur_macro.xacro (robot description, xacro)
@@ -374,4 +374,28 @@
       <child link="${tf_prefix}tool0"/>
     </joint>
+    <link name="cylinder_link">
+      <visual>
+        <geometry>
+          <cylinder length="0.05" radius="0.05"/>
+        </geometry>
+        <material name="blue">
+          <color rgba="0.0 0.0 1.0 1.0"/>
+        </material>
+      </visual>
+      <collision>
+        <geometry>
+          <cylinder length="0.05" radius="0.05"/>
+        </geometry>
+      </collision>
+      <inertial>
+        <mass value="1.0"/>
+        <inertia ixx="0.005" ixy="0.0" ixz="0.0" iyy="0.005" iyz="0.0" izz="0.005"/>
+      </inertial>
+    </link>
+    <joint name="wrist_3_link-fixed_joint" type="fixed">
+      <parent link="wrist_3_link"/>
+      <child link="cylinder_link"/>
+      <origin rpy="0 0 0" xyz="0 0 ${wrist_3_inertia_length -0.014}"/>
+    </joint>
   </xacro:macro>
 </robot>

Commit message: Added table for collisions

File: src/Universal_Robots_ROS2_Description/urdf/ur_macro.xacro (robot description, xacro)
@@ -398,4 +398,28 @@
       <origin rpy="0 0 0" xyz="0 0 ${wrist_3_inertia_length -0.014}"/>
     </joint>
+<link name="table">
+  <visual>
+    <geometry>
+      <box size="0.2 0.2 0.5"/>
+    </geometry>
+    <material name="red">
+      <color rgba="0.0 1.0 0.0 1.0"/>
+    </material>
+  </visual>
+  <collision>
+    <geometry>
+      <box size="0.2 0.2 0.5"/>
+    </geometry>
+  </collision>
+  <inertial>
+    <mass value="1.0"/>
+    <inertia ixx="0.005" ixy="0.0" ixz="0.0" iyy="0.005" iyz="0.0" izz="0.005"/>
+  </inertial>
+</link>
+<joint name="${tf_prefix}base_link-${tf_prefix}base" type="fixed">
+  <parent link="${tf_prefix}base_link"/>
+  <child link="table"/>
+  <origin xyz="0 0 -0.251" rpy="0 0 0"/>
+</joint>
   </xacro:macro>
 </robot>

Commit message: bigger table + depth implemented

File: src/Universal_Robots_ROS2_Description/urdf/ur_macro.xacro (robot description, xacro)
@@ -401,5 +401,5 @@
   <visual>
     <geometry>
-      <box size="0.2 0.2 0.5"/>
+      <box size="0.3 0.3 0.5"/>
     </geometry>
     <material name="red">
@@ -409,5 +409,5 @@
   <collision>
     <geometry>
-      <box size="0.2 0.2 0.5"/>
+      <box size="0.3 0.3 0.5"/>
     </geometry>
   </collision>

Commit message: Debuging strange movements

File: src/Universal_Robots_ROS2_Description/urdf/ur_macro.xacro (robot description, xacro)
@@ -401,5 +401,5 @@
   <visual>
     <geometry>
-      <box size="0.3 0.3 0.5"/>
+      <box size="0.25 0.25 0.5"/>
     </geometry>
     <material name="red">
@@ -409,5 +409,5 @@
   <collision>
     <geometry>
-      <box size="0.3 0.3 0.5"/>
+      <box size="0.25 0.25 0.5"/>
     </geometry>
   </collision>

Commit message: more logs, shrinked table

File: src/Universal_Robots_ROS2_Description/urdf/ur_macro.xacro (robot description, xacro)
@@ -401,5 +401,5 @@
   <visual>
     <geometry>
-      <box size="0.25 0.25 0.5"/>
+      <box size="0.2 0.2 0.5"/>
     </geometry>
     <material name="red">
@@ -409,5 +409,5 @@
   <collision>
     <geometry>
-      <box size="0.25 0.25 0.5"/>
+      <box size="0.2 0.2 0.5"/>
     </geometry>
   </collision>

Commit message: changed urdf

File: src/Universal_Robots_ROS2_Description/urdf/ur_macro.xacro (robot description, xacro)
@@ -370,5 +370,5 @@
     <joint name="${tf_prefix}flange-tool0" type="fixed">
       <!-- default toolframe - X+ left, Y+ up, Z+ front -->
-      <origin xyz="0 0 0" rpy="${pi/2.0} 0 ${pi/2.0}"/>
+      <origin xyz="0.19 0 0" rpy="${pi/2.0} 0 ${pi/2.0}"/>
       <parent link="${tf_prefix}flange"/>
       <child link="${tf_prefix}tool0"/>
@@ -377,5 +377,5 @@
       <visual>
         <geometry>
-          <cylinder length="0.05" radius="0.05"/>
+          <cylinder length="0.19" radius="0.05"/>
         </geometry>
         <material name="blue">
@@ -385,5 +385,5 @@
       <collision>
         <geometry>
-          <cylinder length="0.05" radius="0.05"/>
+          <cylinder length="0.19" radius="0.05"/>
         </geometry>
       </collision>
@@ -396,5 +396,5 @@
       <parent link="wrist_3_link"/>
       <child link="cylinder_link"/>
-      <origin rpy="0 0 0" xyz="0 0 ${wrist_3_inertia_length -0.014}"/>
+      <origin rpy="0 0 0" xyz="0 0 ${(wrist_3_inertia_length / 2) + 0.078}"/>
     </joint>
 <link name="table">
